Commit message: Add Unity control tasks and enhance motor node with connection monitoring and odometry support

File: robot.urdf (robot description, URDF)
Before this commit: robot simple_robot, 3 links, 2 joints
Links:
- removed link left_wheel
- removed link right_wheel
- added link cabin; visual box size=0.4 0.35 0.15
- added link front_left_wheel; visual cylinder length=0.08 radius=0.1
- added link front_right_wheel; visual cylinder length=0.08 radius=0.1
- added link headlight_left; visual sphere radius=0.03
- added link headlight_right; visual sphere radius=0.03
- added link rear_left_wheel; visual cylinder length=0.08 radius=0.1
- added link rear_right_wheel; visual cylinder length=0.08 radius=0.1
- link base_link: geometry visual box size=0.4 0.4 0.15
Joints:
- removed joint left_wheel_joint
- removed joint right_wheel_joint
- added joint cabin_joint: type fixed, parent base_link, child cabin, origin xyz=0 0 0.225
- added joint front_left_wheel_joint: type continuous, parent base_link, child front_left_wheel, origin xyz=0.2 0.25 0 rpy=1.5708 0 0, axis 0 0 1
- added joint front_right_wheel_joint: type continuous, parent base_link, child front_right_wheel, origin xyz=0.2 -0.25 0 rpy=1.5708 0 0, axis 0 0 1
- added joint headlight_left_joint: type fixed, parent base_link, child headlight_left, origin xyz=0.3 0.15 0.05
- added joint headlight_right_joint: type fixed, parent base_link, child headlight_right, origin xyz=0.3 -0.15 0.05
- added joint rear_left_wheel_joint: type continuous, parent base_link, child rear_left_wheel, origin xyz=-0.1 0.25 0 rpy=1.5708 0 0, axis 0 0 1
- added joint rear_right_wheel_joint: type continuous, parent base_link, child rear_right_wheel, origin xyz=-0.1 -0.25 0 rpy=1.5708 0 0, axis 0 0 1

Commit message: Refactor robot.urdf for a simplified car model and update DETECT package documentation
- Changed robot name from "car_robot" to "simple_car" in robot.urdf
- Modified car body dimensions for better representation
- Removed cabin and headlight components to streamline the model
- Adjusted wheel dimensions and positions for improved accuracy
- Added comprehensive DETECT package guide in Turkish, covering system architecture, node responsibilities, quick start, driving modes, topics, configuration, troubleshooting, advanced usage, performance optimization, and support information.

File: robot.urdf (robot description, URDF)
Before this commit: robot car_robot, 8 links, 7 joints
Links:
- removed link cabin
- removed link headlight_left
- removed link headlight_right
- link base_link: geometry visual box size=1.26 1.13 0.52
- link front_left_wheel: geometry visual cylinder length=0.05 radius=0.08
- link front_right_wheel: geometry visual cylinder length=0.05 radius=0.08
- link rear_left_wheel: geometry visual cylinder length=0.05 radius=0.08
- link rear_right_wheel: geometry visual cylinder length=0.05 radius=0.08
Joints:
- removed joint cabin_joint
- removed joint headlight_left_joint
- removed joint headlight_right_joint
- joint front_left_wheel_joint: origin xyz=0.2 0.25 0 rpy=1.5708 0 0 -> xyz=0.15 0.15 0 rpy=1.5708 0 0
- joint front_right_wheel_joint: origin xyz=0.2 -0.25 0 rpy=1.5708 0 0 -> xyz=0.15 -0.15 0 rpy=1.5708 0 0
- joint rear_left_wheel_joint: origin xyz=-0.1 0.25 0 rpy=1.5708 0 0 -> xyz=-0.15 0.15 0 rpy=1.5708 0 0
- joint rear_right_wheel_joint: origin xyz=-0.1 -0.25 0 rpy=1.5708 0 0 -> xyz=-0.15 -0.15 0 rpy=1.5708 0 0
